Commit message: added online url
online url

File: urdf/link5_2_online.urdf (robot description, URDF)
Before this commit: robot link5, 9 links, 8 joints
Links:
- removed link link5/base_link
- removed link link5/base_link_inertia
- removed link link5/sensor_0
- removed link link5/sensor_1
- removed link link5/sensor_2
- removed link link5/sensor_3
- removed link link5/sensor_4
- removed link link5/sensor_5
- removed link link5/sensor_6
- added link calibration_link5/base_link
- added link calibration_link5/base_link_inertia; visual mesh filename=https://cdn.jsdelivr.net/gh/cKohl10/gentact_ros_tools@main/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 scale=1 1 1
- added link calibration_link5/sensor_0; collision sphere radius=0.021; visual sphere radius=0.021
- added link calibration_link5/sensor_1; collision sphere radius=0.023; visual sphere radius=0.023
- added link calibration_link5/sensor_2; collision sphere radius=0.022; visual sphere radius=0.022
- added link calibration_link5/sensor_3; collision sphere radius=0.018; visual sphere radius=0.018
- added link calibration_link5/sensor_4; collision sphere radius=0.02; visual sphere radius=0.02
- added link calibration_link5/sensor_5; collision sphere radius=0.022; visual sphere radius=0.022
- added link calibration_link5/sensor_6; collision sphere radius=0.018; visual sphere radius=0.018
Joints:
- removed joint link5/base_joint
- removed joint link5/sensor_0_joint
- removed joint link5/sensor_1_joint
- removed joint link5/sensor_2_joint
- removed joint link5/sensor_3_joint
- removed joint link5/sensor_4_joint
- removed joint link5/sensor_5_joint
- removed joint link5/sensor_6_joint
- added joint calibration_link5/base_joint: type fixed, parent calibration_link5/base_link, child calibration_link5/base_link_inertia, origin xyz=0 0 0 rpy=0 0 0
- added joint calibration_link5/sensor_0_joint: type fixed, parent calibration_link5/base_link, child calibration_link5/sensor_0, origin xyz=0.034 0.127 -0.019 rpy=1.856 -0.000 2.558, axis 0.529 0.801 -0.281
- added joint calibration_link5/sensor_1_joint: type fixed, parent calibration_link5/base_link, child calibration_link5/sensor_1, origin xyz=-0.004 0.118 -0.089 rpy=-1.403 3.142 0.049, axis -0.049 0.985 -0.167
- added joint calibration_link5/sensor_2_joint: type fixed, parent calibration_link5/base_link, child calibration_link5/sensor_2, origin xyz=-0.017 0.107 -0.138 rpy=1.754 0.000 -2.905, axis -0.23 0.956 -0.182
- added joint calibration_link5/sensor_3_joint: type fixed, parent calibration_link5/base_link, child calibration_link5/sensor_3, origin xyz=-0.035 0.129 -0.011 rpy=1.772 -0.000 -2.583, axis -0.519 0.831 -0.2
- added joint calibration_link5/sensor_4_joint: type fixed, parent calibration_link5/base_link, child calibration_link5/sensor_4, origin xyz=-0.008 0.136 0.024 rpy=1.135 -0.000 -3.039, axis -0.093 0.902 0.423
- added joint calibration_link5/sensor_5_joint: type fixed, parent calibration_link5/base_link, child calibration_link5/sensor_5, origin xyz=-0.000 0.099 -0.185 rpy=-1.262 3.142 0.019, axis -0.018 0.952 -0.304
- added joint calibration_link5/sensor_6_joint: type fixed, parent calibration_link5/base_link, child calibration_link5/sensor_6, origin xyz=-0.007 0.130 -0.039 rpy=-1.229 3.142 0.054, axis -0.051 0.941 -0.335
