Commit message: updated_urdf

File: urdf/fr3_plate.urdf (robot description, URDF)
Before this commit: robot fr3, 20 links, 19 joints
Links:
- link fr3_hand: geometry collision mesh filename=package://franka_description/meshes/robot_ee/franka_hand_wh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; visual mesh filename=package://gentact_ros_tools/meshes/end_effectors/large_plat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
- link fr3_link0: geometry collision mesh filename=package://franka_description/meshes/robot_arms/fr3/collisio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; visual mesh filename=https://cdn.jsdelivr.net/gh/frankarobotics/franka_descripti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

File: urdf/link5_2_calibration.urdf (robot description, URDF)
Before this commit: robot link5, 9 links, 8 joints
Links:
- link calibration_link5/base_link_inertia: geometry visual mesh filename=package://gentact_ros_tools/meshes/skin/link5_2.stl scale=1 1 1

Commit message: Updated Viz

File: urdf/fr3_plate.urdf (robot description, URDF)
Before this commit: robot fr3, 20 links, 19 joints
Links:
- link fr3_link0: geometry collision mesh filename=https://cdn.jsdelivr.net/gh/frankarobotics/franka_descripti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; visual mesh filename=https://cdn.jsdelivr.net/gh/frankarobotics/franka_descripti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
- link fr3_link1: geometry collision mesh filename=https://cdn.jsdelivr.net/gh/frankarobotics/franka_descripti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; visual mesh filename=https://cdn.jsdelivr.net/gh/frankarobotics/franka_descripti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

Commit message: changes

File: urdf/fr3_plate.urdf (robot description, URDF)
Before this commit: robot fr3, 20 links, 19 joints
Links:
- link fr3_link5/base_link_inertia: geometry visual mesh filename=package://gentact_ros_tools/meshes/skin/link5_2.stl scale=1 1 1

Commit message: Added fr3 meshes

File: urdf/fr3_plate.urdf (robot description, URDF)
Before this commit: robot fr3, 20 links, 19 joints
Links:
- link fr3_hand: geometry collision mesh filename=package://gentact_ros_tools/meshes/end_effectors/large_plat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; visual mesh filename=package://gentact_ros_tools/meshes/end_effectors/large_plat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
- link fr3_link0: geometry collision mesh filename=package://gentact_ros_tools/meshes/robot_arms/fr3/collision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; visual mesh filename=package://gentact_ros_tools/meshes/robot_arms/fr3/visual/li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
- link fr3_link1: geometry collision mesh filename=package://gentact_ros_tools/meshes/robot_arms/fr3/collision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; visual mesh filename=package://gentact_ros_tools/meshes/robot_arms/fr3/visual/li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
- link fr3_link2: geometry collision mesh filename=package://gentact_ros_tools/meshes/robot_arms/fr3/collision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; visual mesh filename=package://gentact_ros_tools/meshes/robot_arms/fr3/visual/li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
- link fr3_link3: geometry collision mesh filename=package://gentact_ros_tools/meshes/robot_arms/fr3/collision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; visual mesh filename=package://gentact_ros_tools/meshes/robot_arms/fr3/visual/li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
- link fr3_link4: geometry collision mesh filename=package://gentact_ros_tools/meshes/robot_arms/fr3/collision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; visual mesh filename=package://gentact_ros_tools/meshes/robot_arms/fr3/visual/li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
- link fr3_link5: geometry collision mesh filename=package://gentact_ros_tools/meshes/robot_arms/fr3/collision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; visual mesh filename=package://gentact_ros_tools/meshes/robot_arms/fr3/visual/li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
- link fr3_link6: geometry collision mesh filename=package://gentact_ros_tools/meshes/robot_arms/fr3/collision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; visual mesh filename=package://gentact_ros_tools/meshes/robot_arms/fr3/visual/li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
- link fr3_link7: geometry collision mesh filename=package://gentact_ros_tools/meshes/robot_arms/fr3/collision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; visual mesh filename=package://gentact_ros_tools/meshes/robot_arms/fr3/visual/li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
