Commit message: editted viz

File: urdf/fr3_plate_rviz.urdf (robot description, URDF)
Before this commit: robot fr3, 20 links, 19 joints
Links:
- added link fr3_link5/sensor_7; collision sphere radius=0.002; visual sphere radius=0.002
- link fr3_hand: geometry collision mesh filename=file:///home/caleb/ros2_ws/src/gentact_ros_tools/meshes/end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; visual mesh filename=file:///home/caleb/ros2_ws/src/gentact_ros_tools/meshes/end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
- link fr3_link0: geometry collision mesh filename=file:///home/caleb/ros2_ws/src/gentact_ros_tools/meshes/rob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; visual mesh filename=file:///home/caleb/ros2_ws/src/gentact_ros_tools/meshes/rob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
- link fr3_link1: geometry collision mesh filename=file:///home/caleb/ros2_ws/src/gentact_ros_tools/meshes/rob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; visual mesh filename=file:///home/caleb/ros2_ws/src/gentact_ros_tools/meshes/rob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
- link fr3_link2: geometry collision mesh filename=file:///home/caleb/ros2_ws/src/gentact_ros_tools/meshes/rob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; visual mesh filename=file:///home/caleb/ros2_ws/src/gentact_ros_tools/meshes/rob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
- link fr3_link3: geometry collision mesh filename=file:///home/caleb/ros2_ws/src/gentact_ros_tools/meshes/rob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; visual mesh filename=file:///home/caleb/ros2_ws/src/gentact_ros_tools/meshes/rob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
- link fr3_link4: geometry collision mesh filename=file:///home/caleb/ros2_ws/src/gentact_ros_tools/meshes/rob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; visual mesh filename=file:///home/caleb/ros2_ws/src/gentact_ros_tools/meshes/rob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
- link fr3_link5: geometry collision mesh filename=file:///home/caleb/ros2_ws/src/gentact_ros_tools/meshes/rob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; visual mesh filename=file:///home/caleb/ros2_ws/src/gentact_ros_tools/meshes/rob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
- link fr3_link5/base_link_inertia: geometry visual mesh filename=file:///home/caleb/ros2_ws/src/gentact_ros_tools/meshes/ski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 scale=1 1 1
- link fr3_link5/sensor_0: geometry collision sphere radius=0.002; visual sphere radius=0.002
- link fr3_link5/sensor_1: geometry collision sphere radius=0.002; visual sphere radius=0.002
- link fr3_link5/sensor_2: geometry collision sphere radius=0.002; visual sphere radius=0.002
- link fr3_link5/sensor_3: geometry collision sphere radius=0.002; visual sphere radius=0.002
- link fr3_link5/sensor_4: geometry collision sphere radius=0.002; visual sphere radius=0.002
- link fr3_link5/sensor_5: geometry collision sphere radius=0.002; visual sphere radius=0.002
- link fr3_link5/sensor_6: geometry collision sphere radius=0.002; visual sphere radius=0.002
- link fr3_link6: geometry collision mesh filename=file:///home/caleb/ros2_ws/src/gentact_ros_tools/meshes/rob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; visual mesh filename=file:///home/caleb/ros2_ws/src/gentact_ros_tools/meshes/rob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
- link fr3_link7: geometry collision mesh filename=file:///home/caleb/ros2_ws/src/gentact_ros_tools/meshes/rob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; visual mesh filename=file:///home/caleb/ros2_ws/src/gentact_ros_tools/meshes/rob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
Joints:
- added joint fr3_link5/sensor_7_joint: type fixed, parent fr3_link5/base_link, child fr3_link5/sensor_7, origin xyz=-0.019 0.034 0.054 rpy=-0.002 -0.376 0.0, axis -0.367 0.002 0.93
- joint fr3_link5/sensor_0_joint: axis 0.529 0.801 -0.281 -> -0.045 -0.002 0.999; origin xyz=0.034 0.127 -0.019 rpy=1.856 -0.000 2.558 -> xyz=0.0 -0.064 0.054 rpy=0.002 -0.045 0.0
- joint fr3_link5/sensor_1_joint: axis -0.049 0.985 -0.167 -> -0.039 0.084 0.996; origin xyz=-0.004 0.118 -0.089 rpy=-1.403 3.142 0.049 -> xyz=-0.002 -0.105 0.058 rpy=-0.084 -0.039 0.002
- joint fr3_link5/sensor_2_joint: axis -0.23 0.956 -0.182 -> -0.045 -0.031 0.998; origin xyz=-0.017 0.107 -0.138 rpy=1.754 0.000 -2.905 -> xyz=-0.002 -0.022 0.055 rpy=0.031 -0.045 -0.001
- joint fr3_link5/sensor_3_joint: axis -0.519 0.831 -0.2 -> 0.379 -0.002 0.925; origin xyz=-0.035 0.129 -0.011 rpy=1.772 -0.000 -2.583 -> xyz=0.023 0.033 0.052 rpy=0.002 0.389 0.0
- joint fr3_link5/sensor_4_joint: axis -0.093 0.902 0.423 -> 0.866 -0.368 0.34; origin xyz=-0.008 0.136 0.024 rpy=1.135 -0.000 -3.039 -> xyz=0.047 -0.133 0.026 rpy=0.825 1.046 0.494
- joint fr3_link5/sensor_5_joint: axis -0.018 0.952 -0.304 -> 0.049 0.408 0.912; origin xyz=-0.000 0.099 -0.185 rpy=-1.262 3.142 0.019 -> xyz=0.003 0.098 0.043 rpy=0.421 -0.049 0.01
- joint fr3_link5/sensor_6_joint: axis -0.051 0.941 -0.335 -> -0.097 -0.783 0.615; origin xyz=-0.007 0.130 -0.039 rpy=-1.229 3.142 0.054 -> xyz=-0.004 -0.155 0.044 rpy=0.905 -0.097 -0.047
- joint fr3_link5_to_base_link: origin xyz=0 0 0 rpy=0 0 0 -> xyz=0 0.07 -0.08  rpy=1.4 3.14 3.14

Commit message: Working visualizations for spad and self cap

File: urdf/fr3_plate_rviz.urdf (robot description, URDF)
Before this commit: robot fr3, 21 links, 20 joints
Links:
- link fr3_link5/sensor_0: geometry collision sphere radius=0.005; visual sphere radius=0.005
- link fr3_link5/sensor_1: geometry collision sphere radius=0.005; visual sphere radius=0.005
- link fr3_link5/sensor_2: geometry collision sphere radius=0.005; visual sphere radius=0.005
- link fr3_link5/sensor_3: geometry collision sphere radius=0.005; visual sphere radius=0.005
- link fr3_link5/sensor_4: geometry collision sphere radius=0.005; visual sphere radius=0.005
- link fr3_link5/sensor_5: geometry collision sphere radius=0.005; visual sphere radius=0.005
- link fr3_link5/sensor_6: geometry collision sphere radius=0.005; visual sphere radius=0.005
- link fr3_link5/sensor_7: geometry collision sphere radius=0.005; visual sphere radius=0.005
Joints:
- joint fr3_link5_to_base_link: origin xyz=0 0.07 -0.08  rpy=1.4 3.14 3.14 -> xyz=0 0.07 -0.107  rpy=1.4 3.14 3.14

File: urdf/link5_spad.xacro (robot description, xacro)
@@ -11,5 +11,5 @@
   <xacro:property name="sensor_radius" value="0.005" /> <!-- [m] -->
   <!-- Included URDF Files -->
-  <xacro:include filename="$(find gentact_ros_tools_fp)/urdf/self-cap-base.xacro" />
+  <xacro:include filename="$(find gentact_ros_tools)/urdf/self-cap-base.xacro" />
   <!-- Instantiate dermis once -->
   <xacro:dermis_base_macro
