Commit message: made franka link6 urdf

File: urdf/fr3_link6.urdf (robot description, URDF)
Before this commit: robot fr3, 19 links, 18 joints
Links:
- removed link fr3_link6/base_link
- removed link fr3_link6/base_link_inertia
- removed link fr3_link6/sensor_0
- removed link fr3_link6/sensor_1
- removed link fr3_link6/sensor_2
- removed link fr3_link6/sensor_3
- removed link fr3_link6/sensor_4
- removed link fr3_link6/sensor_5
- removed link fr3_link6/sensor_6
- removed link fr3_link6/sensor_7
- added link fr3_link6_sensor_0; collision sphere radius=0.003; visual sphere radius=0.003
- added link fr3_link6_sensor_1; collision sphere radius=0.003; visual sphere radius=0.003
- added link fr3_link6_sensor_2; collision sphere radius=0.003; visual sphere radius=0.003
- added link fr3_link6_sensor_3; collision sphere radius=0.003; visual sphere radius=0.003
- added link fr3_link6_sensor_4; collision sphere radius=0.003; visual sphere radius=0.003
- added link fr3_link6_sensor_5; collision sphere radius=0.003; visual sphere radius=0.003
- added link fr3_link6_sensor_6; collision sphere radius=0.003; visual sphere radius=0.003
- added link fr3_link6_sensor_7; collision sphere radius=0.003; visual sphere radius=0.003
- added link fr3_link6_skin
- added link fr3_link6_skin_inertia; visual mesh filename=package://gentact_ros_tools/meshes/skin/link6_fancy.stl scale=1 1 1
Joints:
- removed joint fr3_link6/base_joint
- removed joint fr3_link6/sensor_0_joint
- removed joint fr3_link6/sensor_1_joint
- removed joint fr3_link6/sensor_2_joint
- removed joint fr3_link6/sensor_3_joint
- removed joint fr3_link6/sensor_4_joint
- removed joint fr3_link6/sensor_5_joint
- removed joint fr3_link6/sensor_6_joint
- removed joint fr3_link6/sensor_7_joint
- removed joint fr3_link6_to_base_link
- added joint fr3_link6_base_joint: type fixed, parent fr3_link6, child fr3_link6_skin, origin xyz=0 0 0 rpy=0 0 0
- added joint fr3_link6_sensor_0_joint: type fixed, parent fr3_link6_skin, child fr3_link6_sensor_0, origin xyz=0.117 -0.045 -0.004 rpy=1.582 0.000 0.494, axis 0.474 -0.881 -0.011
- added joint fr3_link6_sensor_1_joint: type fixed, parent fr3_link6_skin, child fr3_link6_sensor_1, origin xyz=0.133 -0.025 0.039 rpy=1.451 0.000 1.101, axis 0.885 -0.449 0.12
- added joint fr3_link6_sensor_2_joint: type fixed, parent fr3_link6_skin, child fr3_link6_sensor_2, origin xyz=0.140 -0.002 0.030 rpy=1.487 -0.000 1.464, axis 0.991 -0.106 0.084
- added joint fr3_link6_sensor_3_joint: type fixed, parent fr3_link6_skin, child fr3_link6_sensor_3, origin xyz=0.113 0.047 0.002 rpy=1.585 -0.000 2.644, axis 0.477 0.879 -0.015
- added joint fr3_link6_sensor_4_joint: type fixed, parent fr3_link6_skin, child fr3_link6_sensor_4, origin xyz=0.132 0.029 0.018 rpy=1.533 -0.000 2.048, axis 0.888 0.459 0.037
- added joint fr3_link6_sensor_5_joint: type fixed, parent fr3_link6_skin, child fr3_link6_sensor_5, origin xyz=0.141 -0.001 -0.002 rpy=1.581 -0.000 1.470, axis 0.995 -0.1 -0.01
- added joint fr3_link6_sensor_6_joint: type fixed, parent fr3_link6_skin, child fr3_link6_sensor_6, origin xyz=0.130 -0.033 0.015 rpy=1.541 -0.000 0.888, axis 0.776 -0.631 0.03
- added joint fr3_link6_sensor_7_joint: type fixed, parent fr3_link6_skin, child fr3_link6_sensor_7, origin xyz=0.087 0.051 0.036 rpy=1.488 0.000 -3.049, axis -0.092 0.992 0.083
- added joint fr3_link6_skin_joint: type fixed, parent fr3_link6_skin, child fr3_link6_skin_inertia, origin xyz=0 0 0 rpy=0 0 0

File: urdf/link6.urdf (robot description, URDF)
Before this commit: robot link6, 10 links, 9 joints
Links:
- removed link fr3_link6/base_link
- removed link fr3_link6/base_link_inertia
- removed link fr3_link6/sensor_0
- removed link fr3_link6/sensor_1
- removed link fr3_link6/sensor_2
- removed link fr3_link6/sensor_3
- removed link fr3_link6/sensor_4
- removed link fr3_link6/sensor_5
- removed link fr3_link6/sensor_6
- removed link fr3_link6/sensor_7
- added link fr3_link6_sensor_0; collision sphere radius=0.0; visual sphere radius=0.0
- added link fr3_link6_sensor_1; collision sphere radius=0.0; visual sphere radius=0.0
- added link fr3_link6_sensor_2; collision sphere radius=0.0; visual sphere radius=0.0
- added link fr3_link6_sensor_3; collision sphere radius=0.0; visual sphere radius=0.0
- added link fr3_link6_sensor_4; collision sphere radius=0.0; visual sphere radius=0.0
- added link fr3_link6_sensor_5; collision sphere radius=0.0; visual sphere radius=0.0
- added link fr3_link6_sensor_6; collision sphere radius=0.0; visual sphere radius=0.0
- added link fr3_link6_sensor_7; collision sphere radius=0.0; visual sphere radius=0.0
- added link fr3_link6_skin
- added link fr3_link6_skin_inertia; visual mesh filename=package://gentact_ros_tools/meshes/skins/link6.stl scale=1 1 1
Joints:
- removed joint fr3_link6/base_joint
- removed joint fr3_link6/sensor_0_joint
- removed joint fr3_link6/sensor_1_joint
- removed joint fr3_link6/sensor_2_joint
- removed joint fr3_link6/sensor_3_joint
- removed joint fr3_link6/sensor_4_joint
- removed joint fr3_link6/sensor_5_joint
- removed joint fr3_link6/sensor_6_joint
- removed joint fr3_link6/sensor_7_joint
- added joint fr3_link6_base_joint: type fixed, parent fr3_link6_skin, child fr3_link6_skin_inertia, origin xyz=0 0 0 rpy=0 0 0
- added joint fr3_link6_sensor_0_joint: type fixed, parent fr3_link6_skin, child fr3_link6_sensor_0, origin xyz=0.117 -0.045 -0.004 rpy=1.582 0.000 0.494, axis 0.474 -0.881 -0.011
- added joint fr3_link6_sensor_1_joint: type fixed, parent fr3_link6_skin, child fr3_link6_sensor_1, origin xyz=0.133 -0.025 0.039 rpy=1.451 0.000 1.101, axis 0.885 -0.449 0.12
- added joint fr3_link6_sensor_2_joint: type fixed, parent fr3_link6_skin, child fr3_link6_sensor_2, origin xyz=0.140 -0.002 0.030 rpy=1.487 -0.000 1.464, axis 0.991 -0.106 0.084
- added joint fr3_link6_sensor_3_joint: type fixed, parent fr3_link6_skin, child fr3_link6_sensor_3, origin xyz=0.113 0.047 0.002 rpy=1.585 -0.000 2.644, axis 0.477 0.879 -0.015
- added joint fr3_link6_sensor_4_joint: type fixed, parent fr3_link6_skin, child fr3_link6_sensor_4, origin xyz=0.132 0.029 0.018 rpy=1.533 -0.000 2.048, axis 0.888 0.459 0.037
- added joint fr3_link6_sensor_5_joint: type fixed, parent fr3_link6_skin, child fr3_link6_sensor_5, origin xyz=0.141 -0.001 -0.002 rpy=1.581 -0.000 1.470, axis 0.995 -0.1 -0.01
- added joint fr3_link6_sensor_6_joint: type fixed, parent fr3_link6_skin, child fr3_link6_sensor_6, origin xyz=0.130 -0.033 0.015 rpy=1.541 -0.000 0.888, axis 0.776 -0.631 0.03
- added joint fr3_link6_sensor_7_joint: type fixed, parent fr3_link6_skin, child fr3_link6_sensor_7, origin xyz=0.087 0.051 0.036 rpy=1.488 0.000 -3.049, axis -0.092 0.992 0.083

File: urdf/link6.xacro (robot description, xacro)
@@ -4,5 +4,5 @@
   <xacro:property name="namespace" value="$(arg namespace)" />
   <xacro:property name="use_mesh_file" value="true" />
-  <xacro:property name="mesh_file" value="package://gentact_ros_tools/meshes/skins/link6.stl" />
+  <xacro:property name="mesh_file" value="package://gentact_ros_tools/meshes/skin/link6.stl" />
   <xacro:property name="mass" value="0.3" /> <!-- [kg] -->
   <xacro:property name="body_width" value="0.3" /> <!-- [m] -->
@@ -29,5 +29,5 @@
   <xacro:self_cap_sensor
     robot_namespace="${namespace}"
-    parent="${namespace}/base_link"
+    parent="${namespace}_skin"
     sensor_number="0"
     sensor_radius="0.0"
@@ -40,5 +40,5 @@
   <xacro:self_cap_sensor
     robot_namespace="${namespace}"
-    parent="${namespace}/base_link"
+    parent="${namespace}_skin"
     sensor_number="1"
     sensor_radius="0.0"
@@ -51,5 +51,5 @@
   <xacro:self_cap_sensor
     robot_namespace="${namespace}"
-    parent="${namespace}/base_link"
+    parent="${namespace}_skin"
     sensor_number="2"
     sensor_radius="0.0"
@@ -62,5 +62,5 @@
   <xacro:self_cap_sensor
     robot_namespace="${namespace}"
-    parent="${namespace}/base_link"
+    parent="${namespace}_skin"
     sensor_number="3"
     sensor_radius="0.0"
@@ -73,5 +73,5 @@
   <xacro:self_cap_sensor
     robot_namespace="${namespace}"
-    parent="${namespace}/base_link"
+    parent="${namespace}_skin"
     sensor_number="4"
     sensor_radius="0.0"
@@ -84,5 +84,5 @@
   <xacro:self_cap_sensor
     robot_namespace="${namespace}"
-    parent="${namespace}/base_link"
+    parent="${namespace}_skin"
     sensor_number="5"
     sensor_radius="0.0"
@@ -95,5 +95,5 @@
   <xacro:self_cap_sensor
     robot_namespace="${namespace}"
-    parent="${namespace}/base_link"
+    parent="${namespace}_skin"
     sensor_number="6"
     sensor_radius="0.0"
@@ -106,5 +106,5 @@
   <xacro:self_cap_sensor
     robot_namespace="${namespace}"
-    parent="${namespace}/base_link"
+    parent="${namespace}_skin"
     sensor_number="7"
     sensor_radius="0.0"

File: urdf/self-cap-base.xacro (robot description, xacro)
@@ -4,11 +4,11 @@
   <xacro:macro name="dermis_base_macro"
     params="robot_namespace mass body_width body_height use_mesh_file mesh_file *inertia">
-    <link name="${robot_namespace}/base_link"></link>
-    <joint name="${robot_namespace}/base_joint" type="fixed">
+    <link name="${robot_namespace}_skin"></link>
+    <joint name="${robot_namespace}_base_joint" type="fixed">
       <origin xyz="0 0 0" rpy="0 0 0" />
-      <parent link="${robot_namespace}/base_link" />
-      <child link="${robot_namespace}/base_link_inertia" />
+      <parent link="${robot_namespace}_skin" />
+      <child link="${robot_namespace}_skin_inertia" />
     </joint>
-    <link name="${robot_namespace}/base_link_inertia">
+    <link name="${robot_namespace}_skin_inertia">
       <visual>
         <origin xyz="0 0 0" rpy="0 0 0" />
@@ -27,11 +27,11 @@
   <xacro:macro name="self_cap_sensor"
     params="robot_namespace parent sensor_number sensor_radius sensor_length normal_x normal_y normal_z *origin">
-    <joint name="${robot_namespace}/sensor_${sensor_number}_joint" type="fixed">
+    <joint name="${robot_namespace}_sensor_${sensor_number}_joint" type="fixed">
       <xacro:insert_block name="origin" />
       <axis xyz="${normal_x} ${normal_y} ${normal_z}" />
       <parent link="${parent}" />
-      <child link="${robot_namespace}/sensor_${sensor_number}" />
+      <child link="${robot_namespace}_sensor_${sensor_number}" />
     </joint>
-    <link name="${robot_namespace}/sensor_${sensor_number}">
+    <link name="${robot_namespace}_sensor_${sensor_number}">
       <visual>
         <geometry>

Commit message: Rotated sensor

File: urdf/fr3_link6.urdf (robot description, URDF)
Before this commit: robot fr3, 19 links, 18 joints
Joints:
- joint fr3_joint6: origin xyz=0 0 0 rpy=1.570796326794897 0 0 -> xyz=0 0 0 rpy=-1.570796326794897 0 0

Commit message: rotate

File: urdf/fr3_link6.urdf (robot description, URDF)
Before this commit: robot fr3, 19 links, 18 joints
Joints:
- joint fr3_joint6: origin xyz=0 0 0 rpy=-1.570796326794897 0 0 -> xyz=0 0 0 rpy=1.570796326794897 0 0
- joint fr3_link6_base_joint: origin xyz=0 0 0 rpy=0 0 0 -> xyz=0 0 0 rpy=-1.570796326794897 0 0
