Commit message: Working with docker

File: urdf/skin/link6_big.xacro (robot description, xacro)
@@ -28,5 +28,5 @@
       robot_namespace="${namespace}"
       parent="${namespace}_skin"
-      sensor_number="0"
+      sensor_number="2"
       sensor_radius="${sensor_radius}"
       sensor_length="0.057"
@@ -34,5 +34,5 @@
       normal_y="-0.771"
       normal_z="-0.155">
-      <origin xyz="-0.0631 -0.0491 -0.0215" rpy="1.726 0.000 -0.676" />
+      <origin xyz="-0.0231 -0.0491 -0.0815" rpy="1.726 0.000 -0.676" />
     </xacro:self_cap_sensor>
     <xacro:self_cap_sensor
@@ -45,10 +45,10 @@
       normal_y="-0.709"
       normal_z="0.702">
-      <origin xyz="-0.0353 -0.0490 0.0221" rpy="0.793 0.000 -0.103" />
+      <origin xyz="0.0153 -0.0490 -0.0379" rpy="0.793 0.000 -0.103" />
     </xacro:self_cap_sensor>
     <xacro:self_cap_sensor
       robot_namespace="${namespace}"
       parent="${namespace}_skin"
-      sensor_number="2"
+      sensor_number="4"
       sensor_radius="${sensor_radius}"
       sensor_length="0.060"
@@ -56,5 +56,16 @@
       normal_y="-0.117"
       normal_z="0.014">
-      <origin xyz="0.0913 -0.0053 -0.0027" rpy="1.557 -0.000 1.454" />
+      <origin xyz="0.1313 -0.0053 -0.0527" rpy="1.557 -0.000 1.454" />
+    </xacro:self_cap_sensor>
+    <xacro:self_cap_sensor
+      robot_namespace="${namespace}"
+      parent="${namespace}_skin"
+      sensor_number="0"
+      sensor_radius="${sensor_radius}"
+      sensor_length="0.059"
+      normal_x="0.126"
+      normal_y="-0.992"
+      normal_z="0.008">
+      <origin xyz="0.0478 -0.0561 -0.0628" rpy="1.563 -0.000 0.126" />
     </xacro:self_cap_sensor>
     <xacro:self_cap_sensor
@@ -64,19 +75,8 @@
       sensor_radius="${sensor_radius}"
       sensor_length="0.059"
-      normal_x="0.126"
-      normal_y="-0.992"
-      normal_z="0.008">
-      <origin xyz="0.0078 -0.0561 -0.0028" rpy="1.563 -0.000 0.126" />
-    </xacro:self_cap_sensor>
-    <xacro:self_cap_sensor
-      robot_namespace="${namespace}"
-      parent="${namespace}_skin"
-      sensor_number="4"
-      sensor_radius="${sensor_radius}"
-      sensor_length="0.059"
       normal_x="0.280"
       normal_y="-0.960"
       normal_z="0.023">
-      <origin xyz="0.0575 -0.0444 -0.0024" rpy="1.548 -0.000 0.284" />
+      <origin xyz="0.0975 -0.0444 -0.0624" rpy="1.548 -0.000 0.284" />
     </xacro:self_cap_sensor>
     <xacro:self_cap_sensor
@@ -89,5 +89,5 @@
       normal_y="0.998"
       normal_z="0.042">
-      <origin xyz="0.0466 0.0474 0.0006" rpy="1.529 0.000 3.086" />
+      <origin xyz="0.0866 0.0474 -0.0594" rpy="1.529 0.000 3.086" />
     </xacro:self_cap_sensor>
   </xacro:macro>
