Commit message: added all skins with proper transforms. need to test if sensor positions are correct, and need to figure out how to deal with link5 having 2 different ports (currently being used as one link instead of 2 separate links)

File: urdf/skin/link2_fancy.xacro (robot description, xacro)
@@ -94,5 +94,5 @@
       robot_namespace="${namespace}"
       parent="${namespace}_skin"
-      sensor_number="4"
+      sensor_number="6"
       sensor_radius="${sensor_radius}"
       sensor_length="0.05"

File: urdf/skin/self-cap-base.xacro (robot description, xacro)
@@ -9,5 +9,5 @@
         <geometry>
           <xacro:if value="${use_mesh_file}">
-            <mesh filename="${mesh_file}" scale="1 1 1" />
+            <mesh filename="${mesh_file}" scale="0.001 0.001 0.001" />
           </xacro:if>
           <xacro:unless value="${use_mesh_file}">
@@ -33,14 +33,18 @@
     </joint>
     <link name="${robot_namespace}_sensor_${sensor_number}">
-      <visual>
-        <geometry>
-          <sphere radius="${sensor_radius}" /> <!-- [m] -->
-        </geometry>
-      </visual>
-      <collision>
-        <geometry>
-          <sphere radius="${sensor_radius}" /> <!-- [m] -->
-        </geometry>
-      </collision>
+      <xacro:if value="${sensor_radius > 0.0}">
+        <visual>
+          <geometry>
+            <sphere radius="${sensor_radius}" /> <!-- [m] -->
+          </geometry>
+        </visual>
+      </xacro:if>
+      <xacro:if value="${sensor_radius > 0.0}">
+        <collision>
+          <geometry>
+            <sphere radius="${sensor_radius}" /> <!-- [m] -->
+          </geometry>
+        </collision>
+      </xacro:if>
     </link>
   </xacro:macro>
