Commit message: add raw data publishing

File: urdf/compiled/fr3_hybrid_skin.urdf (robot description, URDF)
Before this commit: robot fr3, 61 links, 60 joints
Joints:
- joint link2_sensor_0_joint: axis 0.723 0.688 -0.056 -> 0.106 0.989 -0.108; origin xyz=0.052 0.111 -0.004 rpy=1.627 -0.000 2.332 -> xyz=0.007 0.136 -0.007 rpy=-1.463 -3.142 -0.106
- joint link2_sensor_1_joint: axis 0.458 0.631 0.627 -> -0.341 0.683 0.646; origin xyz=0.029 0.112 0.042 rpy=0.893 0.000 2.514 -> xyz=-0.024 0.113 0.045 rpy=0.869 -0.000 -2.678
- joint link2_sensor_2_joint: axis 0.106 0.989 -0.108 -> -0.777 0.627 -0.06; origin xyz=0.007 0.136 -0.007 rpy=-1.463 -3.142 -0.106 -> xyz=-0.050 0.113 -0.009 rpy=1.630 -0.000 -2.249
- joint link2_sensor_3_joint: axis 0.222 0.969 0.105 -> 0.723 0.688 -0.056; origin xyz=0.009 0.064 0.131 rpy=1.466 0.000 2.917 -> xyz=0.052 0.111 -0.004 rpy=1.627 -0.000 2.332
- joint link2_sensor_4_joint: axis -0.133 0.605 -0.785 -> 0.458 0.631 0.627; origin xyz=-0.009 0.112 -0.051 rpy=-0.668 -3.142 0.217 -> xyz=0.029 0.112 0.042 rpy=0.893 0.000 2.514
- joint link2_sensor_5_joint: axis -0.341 0.683 0.646 -> 0.222 0.969 0.105; origin xyz=-0.024 0.113 0.045 rpy=0.869 -0.000 -2.678 -> xyz=0.009 0.064 0.131 rpy=1.466 0.000 2.917
- joint link2_sensor_6_joint: axis -0.777 0.627 -0.06 -> -0.133 0.605 -0.785; origin xyz=-0.050 0.113 -0.009 rpy=1.630 -0.000 -2.249 -> xyz=-0.009 0.112 -0.051 rpy=-0.668 -3.142 0.217

File: urdf/skin/hybrid/link5_hybrid_back.xacro (robot description, xacro)
@@ -1,9 +1,9 @@
 <?xml version="1.0"?>
 <robot xmlns:xacro="http://ros.org/wiki/xacro">
-  <!-- Macro definition for link5 pt 2 skin -->
+  <!-- Macro definition for link5 pt 1 skin -->
   <xacro:macro name="link5_back_skin" params="parent namespace">
     <!-- Properties -->
     <xacro:property name="use_mesh_file" value="true" />
-    <xacro:property name="mesh_file" value="package://gentact_ros_tools_hybrid/meshes/skin/hybrid/link5_part2_hybrid_dermis.stl" />
+    <xacro:property name="mesh_file" value="package://gentact_ros_tools_hybrid/meshes/skin/hybrid/link5_part1_hybrid_dermis.stl" />
     <xacro:property name="mass" value="0.3" /> <!-- [kg] -->
     <xacro:property name="body_width" value="0.3" /> <!-- [m] -->

File: urdf/skin/hybrid/link5_hybrid_front.xacro (robot description, xacro)
@@ -1,9 +1,9 @@
 <?xml version="1.0"?>
 <robot xmlns:xacro="http://ros.org/wiki/xacro">
-  <!-- Macro definition for link5 pt 1 skin -->
+  <!-- Macro definition for link5 pt 2 skin -->
   <xacro:macro name="link5_front_skin" params="parent namespace">
     <!-- Properties -->
     <xacro:property name="use_mesh_file" value="true" />
-    <xacro:property name="mesh_file" value="package://gentact_ros_tools_hybrid/meshes/skin/hybrid/link5_part1_hybrid_dermis.stl" />
+    <xacro:property name="mesh_file" value="package://gentact_ros_tools_hybrid/meshes/skin/hybrid/link5_part2_hybrid_dermis.stl" />
     <xacro:property name="mass" value="0.3" /> <!-- [kg] -->
     <xacro:property name="body_width" value="0.3" /> <!-- [m] -->

Commit message: added h1_2 urdf and config file with nick's skin.

File: urdf/compiled/fr3_hybrid_skin.urdf (robot description, URDF)
Before this commit: robot fr3, 61 links, 60 joints
Links:
- link fr3_hand: geometry collision mesh filename=package://gentact_descriptions_hybrid/meshes/robot_ee/frank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; visual mesh filename=package://gentact_descriptions_hybrid/meshes/robot_ee/frank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
- link fr3_leftfinger: geometry collision box size=17.5e-3 15.2e-3 18.5e-3; collision box size=17.5e-3 7e-3 23.5e-3
- link fr3_rightfinger: geometry collision box size=17.5e-3 15.2e-3 18.5e-3; collision box size=17.5e-3 7e-3 23.5e-3
